File: lorawan_e78-868ln22s_minipci.sch (KiCad schematic (older format))
At the start: 7 parts, among them Con1 MiniPci, P1 RF2-03E-T-00-50-G, U8 IP4220CZ6

Commit message: Finalized project
Parts:
- added C3, C4: 100n_50V, Capacitors_Smd_0603:100nF_0603, symbol Capacitors_Smd0603:100n_50V
- added Con2: TC2050-IDC-NL, Tag_Connectors:TC2050-IDC-NL, symbol Tag_Connectors:TC2050-IDC-NL
- added NTC1: NTCS0603E3103FMT, NTC_Thermistors:NTCS0603E3103FMT, symbol NTC_Thermistors:NTCS0603E3103FMT
- added R2, R3, R4, R5: 4k7, Resistor_Smd_0603:4k7_0603, symbol Resistors_Smd0603:4k7
- added R6, R7, R8: 0R, Resistor_Smd_0603:0R_0603, symbol Resistors_Smd0603:0R
- added U1: DS18B20U, Temperature_Sensors:DS18B20U_MSOP-8_3x3mm_P0.65mm, symbol Temperature_Sensors:DS18B20U
- added U2: TCN75A, Temperature_Sensors:TCN75A_SOIC8, symbol Temperature_Sensors:TCN75A
Connections:
- net 3V3: now also C3.1, C4.1, Con2.3 (P3), NTC1.2, R2.1, R3.1, R4.1, U1.8 (VDD), U2.7 (A0), U2.8 (VDD)
- net GND: now also C3.2, C4.2, Con2.4 (P4), R5.2, U1.4 (VSS), U2.4 (VSS), U2.5 (A2), U2.6 (A1)
- net at Module1.22 (SWD_DATA), U8.4 (I/O3): now also Con2.10 (P10), R7.1; no longer Con1.10 (USIM_DATA)
- net at Con1.11 (UART_CTS): now also Module1.20 (UART_RX), U8.1 (I/O1)
- net at Module1.23 (SWD_CLK), U8.6 (I/O4): now also Con2.6 (P6), R8.1; no longer Con1.12 (USIM_CLK)
- net at Con1.13 (UART_RTS): now also Module1.21 (UART_TX), U8.3 (I/O2)
- net at C1.1, Module1.16 (XRES), R1.2: now also Con2.7 (P7), R6.1; no longer Con1.22 (~PERST)
- net at Module1.17 (ADC_IN): now also NTC1.1, R5.1
- net at Module1.4 (DIO1): now also R4.2, U1.1 (DQ)
- net at Module1.6 (I2C_SDA): now also R3.2, U2.1 (SDA)
- net at Module1.7 (I2C_SCL): now also R2.2, U2.2 (SCL)
- net SCL: no longer names the net of Con1.30 (SCL)
- net SDA: no longer names the net of Con1.32 (SDA)
- net UART_GPS_3V3_RXD: no longer names the net of Con1.44 (GPIO0)
- net UART_GPS_3V3_TXD: no longer names the net of Con1.46 (GPIO1)
- new net: Con1.10 (USIM_DATA), R7.2
- new net: Con1.12 (USIM_CLK), R8.2
- new net: Con1.22 (~PERST), R6.2
- now unconnected: Con1.17 (UART_RXD), Con1.19 (UART_TXD)
- no-connect marks 25 -> 29
Other:
- moved on the sheet: C1, C2, Con1, Module1, P1, R1, U8
